File: kicad/serge-r5-triple-wave-shaper.kicad_pcb (KiCad board)
At the start: 2 copper layers, 99.1 x 152.4 mm, 97 parts, among them J1 Banana Socket PanelMount, J11 Conn_01x06_Female, J12 Conn_01x06_Male, J13 Banana Socket PanelMount, J14 Banana Socket PanelMount, J15 Banana Socket PanelMount, J16 Banana Socket PanelMount, J17 Conn_01x06_Female, J18 Conn_01x06_Male, J2 Banana Socket PanelMount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

Commit message: Regenerate gerbers after tweaks
Parts:
- C1, C2, C7: footprint Rumblesan_Standard_Parts:C_Rect_L7.0mm_W3.5mm_P5.00mm -> Capacitor_THT:C_Rect_L7.2mm_W8.5mm_P5.00mm_FKP2_FKP2_MKS2_MKP2
- J20: moved to B.Cu
- SW1, SW2, SW3: footprint Rumblesan_Standard_Parts:Toggle_Switch_100SP1T1B3M2QE -> Rumblesan_Standard_Parts:Toggle_Switch_100SP-M2
- moved J3 117.1 mm to (62.2, 173.4), turned to 180 degrees
- moved J7 117.1 mm to (36.8, 59.1), turned to -90 degrees
- moved J1 114.3 mm to (36.8, 154.3), turned to 180 degrees
- moved J5 114.3 mm to (36.8, 40.0), turned to -90 degrees
- moved J4 95.2 mm to (62.2, 135.3)
- moved J8 95.2 mm to (62.2, 40.0)
- moved J2 95.2 mm to (36.8, 173.4)
- moved J6 95.2 mm to (36.8, 78.1)
- moved R3 85.0 mm to (83.2, 138.6)
- moved D4 82.4 mm to (90.8, 63.6)
- moved R9 81.8 mm to (83.2, 51.7)
- moved D8 79.7 mm to (105.3, 78.9), turned to 180 degrees
- moved C4 79.7 mm to (105.2, 75.6), turned to 180 degrees
- moved D5 79.4 mm to (105.3, 150.5)
- moved C3 79.4 mm to (98.2, 157.0)
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Connections:
- C5 pad 1: Net-(J20-Pin_5) -> Net-(J12-Pin_5)
- C6 pad 1: Net-(J12-Pin_1) -> Net-(J20-Pin_3)
- J1 pad 1: Net-(J21-Pin_8) -> Net-(J11-Pin_3)
- J12 pad 1: Net-(J12-Pin_1) -> Net-(D2-A)
- J12 pad 2: Net-(J12-Pin_2) -> Net-(D1-A)
- J12 pad 5: Net-(D4-A) -> Net-(J12-Pin_5)
- J12 pad 6: Net-(D3-A) -> Net-(J12-Pin_6)
- J2 pad 1: Net-(J21-Pin_4) -> Net-(J11-Pin_2)
- J20 pad 1: GND -> Net-(J20-Pin_1)
- J20 pad 2: GND -> Net-(J20-Pin_2)
- J20 pad 3: Net-(D2-A) -> Net-(J20-Pin_3)
- J20 pad 4: Net-(D1-A) -> Net-(J20-Pin_4)
- J20 pad 5: Net-(J20-Pin_5) -> Net-(D4-A)
- J20 pad 6: Net-(J20-Pin_6) -> Net-(D3-A)
- J20 pad 7: Net-(J20-Pin_7) -> GND
- J20 pad 8: Net-(J20-Pin_8) -> GND
- J21 pad 1: GND -> Net-(J21-Pin_1)
- J21 pad 2: GND -> Net-(J21-Pin_2)
- J21 pad 7: Net-(J21-Pin_7) -> GND
- J21 pad 8: Net-(J21-Pin_8) -> GND
- J3 pad 1: Net-(J21-Pin_3) -> Net-(J11-Pin_1)
- J5 pad 1: Net-(J11-Pin_4) -> Net-(J21-Pin_1)
- J6 pad 1: Net-(J11-Pin_6) -> Net-(J21-Pin_6)
- J7 pad 1: Net-(J11-Pin_5) -> Net-(J21-Pin_5)
- JP1 pad 2: Net-(J20-Pin_8) -> Net-(J12-Pin_3)
- JP1 pad 3: Net-(J20-Pin_5) -> Net-(J12-Pin_5)
- JP2 pad 2: Net-(J12-Pin_4) -> Net-(J20-Pin_1)
- JP2 pad 3: Net-(J12-Pin_1) -> Net-(J20-Pin_3)
- R10 pad 1: Net-(J12-Pin_3) -> Net-(J20-Pin_4)
- R15 pad 2: Net-(J20-Pin_5) -> Net-(J12-Pin_5)
- R17 pad 2: Net-(J12-Pin_1) -> Net-(J20-Pin_3)
- R3 pad 1: Net-(J20-Pin_7) -> Net-(J12-Pin_4)
- R4 pad 1: Net-(J20-Pin_6) -> Net-(J12-Pin_6)
- R9 pad 1: Net-(J12-Pin_2) -> Net-(J20-Pin_2)
- RV1 pad 2: Net-(J21-Pin_7) -> Net-(J21-Pin_2)
- RV1 pad 3: Net-(J4-Pad1) -> Net-(J8-Pad1)
- RV2 pad 2: Net-(J21-Pin_6) -> Net-(J11-Pin_6)
- RV3 pad 2: Net-(J11-Pin_3) -> Net-(J11-Pin_4)
- RV3 pad 3: Net-(J8-Pad1) -> Net-(J4-Pad1)
- RV6 pad 2: Net-(J17-Pin_3) -> Net-(J17-Pin_2)
- SW1 pad 3: Net-(J11-Pin_1) -> Net-(J21-Pin_3)
- SW2 pad 2: Net-(J11-Pin_2) -> Net-(J21-Pin_4)
- SW3 pad 1: Net-(J21-Pin_5) -> Net-(J11-Pin_5)
- SW3 pad 2: Net-(J17-Pin_2) -> Net-(J17-Pin_3)
- U1 pad 10: Net-(R14-Pad2) -> Net-(R13-Pad2)
- U1 pad 11: Net-(D7-A) -> Net-(D5-A)
- U1 pad 12: Net-(D7-K) -> Net-(D5-K)
- U1 pad 2: Net-(D5-K) -> Net-(D7-K)
- U1 pad 3: Net-(D5-A) -> Net-(D7-A)
- U1 pad 4: Net-(R13-Pad2) -> Net-(R14-Pad2)
Routing:
- net Net-(J11-Pin_6): track 32.6 -> 75.7 mm
- net Net-(D5-A): track 35.7 -> 77.6 mm
- net Net-(J21-Pin_7): track 39.1 -> 0.00 mm
- net Net-(J21-Pin_2): track 0.00 -> 37.2 mm
- net Net-(D7-A): track 80.6 -> 43.7 mm
- net Net-(D7-K): track 80.9 -> 53.1 mm
- net Net-(J21-Pin_3): track 10.6 -> 37.7 mm
- net Net-(D5-K): track 40.1 -> 66.5 mm
- net Net-(J21-Pin_6): track 42.0 -> 16.8 mm
- net Net-(J21-Pin_5): track 33.2 -> 9.57 mm
- net Net-(J20-Pin_5): track 22.9 -> 0.00 mm
- net Net-(J17-Pin_4): track 82.7 -> 59.9 mm
- net Net-(J12-Pin_5): track 0.00 -> 22.2 mm
- net Net-(J20-Pin_3): track 0.00 -> 20.9 mm
- net Net-(J21-Pin_4): track 20.1 -> 40.3 mm
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