File: kicad/serge-r5-triple-wave-shaper.kicad_sch (KiCad schematic)
At the start: 90 parts, among them J1 Banana Socket PanelMount, J11 Conn_01x06_Female, J12 Conn_01x06_Male, J13 Banana Socket PanelMount, J14 Banana Socket PanelMount, J15 Banana Socket PanelMount, J16 Banana Socket PanelMount, J17 Conn_01x06_Female, J18 Conn_01x06_Male, J2 Banana Socket PanelMount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

Commit message: Regenerate gerbers after tweaks
Parts:
- C1, C2, C7: footprint Rumblesan_Standard_Parts:C_Rect_L7.0mm_W3.5mm_P5.00mm -> Capacitor_THT:C_Rect_L7.2mm_W8.5mm_P5.00mm_FKP2_FKP2_MKS2_MKP2
- J6: Name WS3 CV2 -> WS3 VC2
- J7: Name WS3 CV1 -> WS3 VC1
- SW1, SW2, SW3: footprint Rumblesan_Standard_Parts:Toggle_Switch_100SP1T1B3M2QE -> Rumblesan_Standard_Parts:Toggle_Switch_100SP-M2
Connections:
- net GND: now also J20.7 (Pin_7), J20.8 (Pin_8), J21.7 (Pin_7), J21.8 (Pin_8); no longer J20.1 (Pin_1), J20.2 (Pin_2), J21.1 (Pin_1), J21.2 (Pin_2)
- net at SW3.1 (A): now also J11.5 (Pin_5); no longer J21.5 (Pin_5)
- net at SW3.2 (B): now also J17.3 (Pin_3); no longer J17.2 (Pin_2)
- net at D3.2 (A), R5.2: now also J20.6 (Pin_6); no longer J12.6 (Pin_6)
- net at C3.1, D5.2 (A), D6.1 (K)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: now also U1.11 (-); no longer U1.3 (-)
- net at J2.1: now also J11.2 (Pin_2); no longer J21.4 (Pin_4)
- net at C6.1, JP2.3 (B), R17.2: now also J20.3 (Pin_3); no longer J12.1 (Pin_1)
- net at J12.2 (Pin_2): now also D1.2 (A), R1.2; no longer R9.1
- net at J12.3 (Pin_3): now also JP1.2 (C); no longer R10.1
- net at J12.4 (Pin_4): now also R3.1; no longer JP2.2 (C)
- net at D4.2 (A), R6.2: now also J20.5 (Pin_5); no longer J12.5 (Pin_5)
- net at J5.1: now also J21.1 (Pin_1); no longer J11.4 (Pin_4)
- net at J7.1: now also J21.5 (Pin_5); no longer J11.5 (Pin_5)
- net at J11.1 (Pin_1): now also J3.1; no longer SW1.3 (C)
- net at SW2.2 (B): now also J21.4 (Pin_4); no longer J11.2 (Pin_2)
- net at J11.3 (Pin_3): now also J1.1; no longer RV3.2
- net at J11.6 (Pin_6): now also RV2.2; no longer J6.1
- net at C1.2, D5.1 (K), R7.2: now also U1.12 (+); no longer U1.2 (+)
- net at R13.2, R15.1, RV4.3: now also U1.10; no longer U1.4
- net at C4.1, D7.2 (A), D8.1 (K)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: now also U1.3 (-); no longer U1.11 (-)
- net at J21.3 (Pin_3): now also SW1.3 (C); no longer J3.1
- net at C2.2, D7.1 (K), R11.2: now also U1.2 (+); no longer U1.12 (+)
- net at RV3.3: now also J4.1; no longer J8.1
- net at R4.1: now also J12.6 (Pin_6); no longer J20.6 (Pin_6)
- net at D2.2 (A), R2.2: now also J12.1 (Pin_1); no longer J20.3 (Pin_3)
- net at RV6.2: now also J17.2 (Pin_2); no longer J17.3 (Pin_3)
- net at RV1.2: now also J21.2 (Pin_2); no longer J21.7 (Pin_7)
- net at RV1.3: now also J8.1; no longer J4.1
- net at C5.1, JP1.3 (B), R15.2: now also J12.5 (Pin_5); no longer J20.5 (Pin_5)
- net at R14.2, R17.1, RV5.3: now also U1.4; no longer U1.10
- net at J21.6 (Pin_6): now also J6.1; no longer RV2.2
- new net: J11.4 (Pin_4), RV3.2
- new net: J20.2 (Pin_2), R9.1
- new net: J20.1 (Pin_1), JP2.2 (C)
- new net: J20.4 (Pin_4), R10.1
Other:
- moved on the sheet: J1, J11, J12, J2, J20, J21, J3, J4, J5, J6, J7, J8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
